File: kicad/m3/v2.2b -ESP32-DevKitC-VIE/TRS-IO-M3.kicad_sch (KiCad schematic)
At the start: 44 parts, among them J1 Conn_02x25_Odd_Even, J2 Conn_02x25_Odd_Even, J3 Conn_01x19, J4 Conn_01x02_Male, J5 Conn_01x06_Male, J6 Conn_01x06_Male, J7 AudioJack3, Q1 2N7002, Q2 2N7002, Q3 2N7002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

Commit message: added gerbers
Parts:
- D1, J2, J3, J4, J5, J6, J7, SW1, U5, U6: now not fitted
Changed lines of the file:
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@@
 		(in_bom yes)
 		(on_board yes)
-		(dnp no)
+		(dnp yes)
 		(property "Reference" "U6"
 			(at 106.68 41.91 0)
@@
 		(in_bom yes)
 		(on_board yes)
-		(dnp no)
+		(dnp yes)
 		(property "Reference" "D1"
 			(at 215.9 132.842 0)
@@
 		(in_bom yes)
 		(on_board yes)
-		(dnp no)
+		(dnp yes)
 		(property "Reference" "SW1"
 			(at 218.44 190.5 0)
@@
 		(in_bom yes)
 		(on_board yes)
-		(dnp no)
+		(dnp yes)
 		(property "Reference" "J4"
 			(at 292.3032 147.8026 0)
@@
 		(in_bom yes)
 		(on_board yes)
-		(dnp no)
+		(dnp yes)
 		(fields_autoplaced yes)
 		(property "Reference" "J3"
@@
 		(in_bom yes)
 		(on_board yes)
-		(dnp no)
+		(dnp yes)
 		(fields_autoplaced yes)
 		(property "Reference" "J2"
@@
 		(in_bom yes)
 		(on_board yes)
-		(dnp no)
+		(dnp yes)
 		(fields_autoplaced yes)
 		(property "Reference" "J6"
@@
 		(in_bom yes)
 		(on_board yes)
-		(dnp no)
+		(dnp yes)
 		(property "Reference" "U5"
 			(at 200.66 40.64 0)
@@
 		(in_bom yes)
 		(on_board yes)
-		(dnp no)
+		(dnp yes)
 		(property "Reference" "J7"
 			(at 338.582 210.3882 0)
@@
 		(in_bom yes)
 		(on_board yes)
-		(dnp no)
+		(dnp yes)
 		(fields_autoplaced yes)
 		(property "Reference" "J5"
